File: hexpansion-devkit.kicad_pcb (KiCad board)
At the start: 4 copper layers, 73.2 x 48 mm, 22 parts, among them J1 Conn_02x10_Counter_Clockwise, J2 Conn_02x10_Counter_Clockwise, J3 Conn_02x10_Counter_Clockwise, J4 Conn_01x07, J5 Conn_02x10_Odd_Even, J6 Conn_02x10_Odd_Even, J7 Conn_02x10_Odd_Even, U1 AW9523B, U2 TCA9548APWR

Commit message: Revision 2
Parts:
- added R3: 4K7, Resistor_SMD:R_0603_1608Metric, F.Cu at (118.1, 63.6)
- added R4: 4K7, Resistor_SMD:R_0603_1608Metric, F.Cu at (116.6, 63.6)
- added R5: 4K7, Resistor_SMD:R_0603_1608Metric, F.Cu at (135.6, 72.4)
- added R6: 4K7, Resistor_SMD:R_0603_1608Metric, F.Cu at (134.1, 72.4)
- R1, R2: value R -> 4k7
- moved R2 0.25 mm to (141.0, 63.5)
Routing:
- net /SDA: track 18.0 -> 32.4 mm
- net /SCL: track 17.2 -> 26.0 mm
- net +3V3: track 93.0 -> 101.4 mm
- net /SYS_SCL: track 23.1 -> 22.4 mm
- net /SYS_SDA: track 19.4 -> 18.8 mm
