File: hexpansion-devkit.kicad_sch (KiCad schematic)
At the start: 21 parts, among them J1 Conn_02x10_Counter_Clockwise, J2 Conn_02x10_Counter_Clockwise, J3 Conn_02x10_Counter_Clockwise, J4 Conn_01x07, J5 Conn_02x10_Odd_Even, J6 Conn_02x10_Odd_Even, J7 Conn_02x10_Odd_Even, U1 AW9523B, U2 TCA9548APWR

Commit message: Revision 2
Parts:
- added R3, R4, R5, R6: 4K7, Resistor_SMD:R_0603_1608Metric, symbol Device:R
- R1, R2: value R -> 4k7; LCSC C2907127 -> C217361
Connections:
- net +3V3: now also R3.1, R4.1, R5.1, R6.1
- net SCL: now also R3.2
- net SDA: now also R4.2
- net SYS_SCL: now also R5.2
- net SYS_SDA: now also R6.2
- no-connect marks 0 -> 9
Other:
- moved on the sheet: C1, C2, R1, R2
