File: pcb/hexpansion-devkit.kicad_pcb (KiCad board)
At the start: 4 copper layers, 73.2 x 48 mm, 26 parts, among them J1 Conn_02x10_Counter_Clockwise, J2 Conn_02x10_Counter_Clockwise, J3 Conn_02x10_Counter_Clockwise, J4 Conn_01x07, J5 Conn_02x10_Odd_Even, J6 Conn_02x10_Odd_Even, J7 Conn_02x10_Odd_Even, U1 AW9523B, U2 TCA9548APWR

Commit message: Tidy PCB silkscreen, add new render
Routing:
- net /SDA: track 32.4 -> 31.2 mm
Other:
- board text added: "3V3"
- board text added: "GND"
- board text added: "INT"
- board text added: "RST"
- board text added: "SCK"
- board text added: "SDA"
- board text added: "i2c"
- board text removed: "I"
- board text removed: "I2C"
- board text removed: "R"
- board text removed: "SL"
Changed lines of the file:
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@@
 	)
 	(gr_line
-		(start 131.318 65.532)
-		(end 131.318 65.278)
+		(start 131.318 65.786)
+		(end 131.318 65.024)
 		(stroke
 			(width 0.1)
@@
 	)
 	(gr_line
-		(start 136.398 65.532)
-		(end 136.398 65.278)
+		(start 136.398 65.786)
+		(end 136.398 65.024)
 		(stroke
 			(width 0.1)
@@
 	)
 	(gr_line
-		(start 135.89 65.532)
-		(end 136.398 65.532)
+		(start 110.49 74.93)
+		(end 110.998 74.93)
 		(stroke
 			(width 0.1)
@@
 	)
 	(gr_line
-		(start 127.508 65.532)
-		(end 126.238 65.532)
+		(start 135.89 65.786)
+		(end 136.398 65.786)
 		(stroke
 			(width 0.1)
@@
 	)
 	(gr_line
-		(start 133.858 65.532)
-		(end 133.858 65.278)
+		(start 140.462 74.93)
+		(end 143.51 74.93)
 		(stroke
 			(width 0.1)
@@
 	)
 	(gr_line
-		(start 126.238 65.532)
-		(end 126.238 65.278)
+		(start 128.27 87.884)
+		(end 128.27 84.836)
 		(stroke
 			(width 0.1)
@@
 	)
 	(gr_line
-		(start 130.048 65.532)
-		(end 131.318 65.532)
+		(start 110.49 77.47)
+		(end 113.538 77.47)
 		(stroke
 			(width 0.1)
@@
 	)
 	(gr_line
-		(start 134.366 65.532)
-		(end 133.858 65.532)
+		(start 110.998 74.93)
+		(end 110.998 77.47)
+		(stroke
+			(width 0.1)
+			(type default)
+		)
+		(layer "F.SilkS")
+	)
+	(gr_line
+		(start 127.762 65.786)
+		(end 126.238 65.786)
+		(stroke
+			(width 0.1)
+			(type default)
+		)
+		(layer "F.SilkS")
+	)
+	(gr_line
+		(start 143.002 77.47)
+		(end 143.002 74.93)
+		(stroke
+			(width 0.1)
+			(type default)
+		)
+		(layer "F.SilkS")
+	)
+	(gr_line
+		(start 133.858 65.786)
+		(end 133.858 65.024)
+		(stroke
+			(width 0.1)
+			(type default)
+		)
+		(layer "F.SilkS")
+	)
+	(gr_line
+		(start 126.238 65.786)
+		(end 126.238 65.024)
+		(stroke
+			(width 0.1)
+			(type default)
+		)
+		(layer "F.SilkS")
+	)
+	(gr_line
+		(start 129.794 65.786)
+		(end 131.318 65.786)
+		(stroke
+			(width 0.1)
+			(type default)
+		)
+		(layer "F.SilkS")
+	)
+	(gr_line
+		(start 143.51 77.47)
+		(end 143.002 77.47)
+		(stroke
+			(width 0.1)
+			(type default)
+		)
+		(layer "F.SilkS")
+	)
+	(gr_line
+		(start 125.73 87.884)
+		(end 125.73 87.376)
+		(stroke
+			(width 0.1)
+			(type default)
+		)
+		(layer "F.SilkS")
+	)
+	(gr_line
+		(start 125.73 87.376)
+		(end 128.27 87.376)
+		(stroke
+			(width 0.1)
+			(type default)
+		)
+		(layer "F.SilkS")
+	)
+	(gr_line
+		(start 134.366 65.786)
+		(end 133.858 65.786)
 		(stroke
 			(width 0.1)
@@
 		)
 	)
-	(gr_text "R"
-		(at 133.858 61.722 0)
+	(gr_text "RST"
+		(at 133.858 61.468 0)
 		(layer "F.SilkS")
 		(effects
 			(font
-				(size 1 1)
+				(size 0.6 0.6)
 				(thickness 0.1)
 			)
@@
 		)
 	)
-	(gr_text "R"
-		(at 131.318 61.722 0)
+	(gr_text "RST"
+		(at 131.318 61.468 0)
 		(layer "F.SilkS")
 		(effects
 			(font
-				(size 1 1)
+				(size 0.6 0.6)
 				(thickness 0.1)
 			)
@@
 		)
 	)
-	(gr_text "SL"
+	(gr_text "SC"
 		(at 125.73 94.488 90)
 		(layer "F.SilkS")
@@
 		(effects
 			(font
-				(size 1 1)
+				(size 0.6 0.6)
 				(thickness 0.1)
 			)
@@
 		(effects
 			(font
-				(size 1 1)
+				(size 0.6 0.6)
 				(thickness 0.1)
 			)
@@
 	)
 	(gr_text "E power"
-		(at 127 85.344 0)
+		(at 124.206 84.074 0)
 		(layer "F.SilkS")
 		(effects
@@
 				(thickness 0.1)
 			)
-			(justify top)
+			(justify right)
 		)
 	)
@@
 		(effects
 			(font
-				(size 1 1)
+				(size 0.6 0.6)
 				(thickness 0.1)
 			)
@@
 		(effects
 			(font
-				(size 1 1)
+				(size 0.6 0.6)
 				(thickness 0.1)
 			)
@@
 		(effects
 			(font
-				(size 1 1)
+				(size 0.6 0.6)
 				(thickness 0.1)
 			)
@@
 		)
 	)
-	(gr_text "SC"
-		(at 126.238 61.722 0)
+	(gr_text "SCK"
+		(at 126.238 61.468 0)
 		(layer "F.SilkS")
 		(effects
 			(font
-				(size 1 1)
+				(size 0.6 0.6)
 				(thickness 0.1)
 			)
@@
 		)
 	)
-	(gr_text "SD"
-		(at 128.778 61.722 0)
+	(gr_text "SDA"
+		(at 128.778 61.468 0)
 		(layer "F.SilkS")
 		(effects
 			(font
-				(size 1 1)
+				(size 0.6 0.6)
 				(thickness 0.1)
 			)
@@
 	)
 	(gr_text "IO"
-		(at 135.128 65.024 0)
+		(at 135.128 65.786 0)
 		(layer "F.SilkS")
 		(effects
 			(font
-				(size 1 1)
+				(size 0.6 0.6)
 				(thickness 0.1)
 			)
-			(justify top)
 		)
 	)
@@
 		)
 	)
-	(gr_text "V"
-		(at 123.698 61.722 0)
+	(gr_text "3V3"
+		(at 123.698 61.468 0)
 		(layer "F.SilkS")
 		(effects
 			(font
-				(size 1 1)
+				(size 0.6 0.6)
 				(thickness 0.1)
 			)
@@
 		(effects
 			(font
-				(size 1 1)
+				(size 0.6 0.6)
 				(thickness 0.1)
 			)
@@
 		(effects
 			(font
-				(size 1 1)
+				(size 0.6 0.6)
 				(thickness 0.1)
 			)
@@
 		)
 	)
-	(gr_text "I"
-		(at 136.398 61.722 0)
+	(gr_text "INT"
+		(at 136.398 61.468 0)
 		(layer "F.SilkS")
 		(effects
 			(font
-				(size 1 1)
+				(size 0.6 0.6)
 				(thickness 0.1)
 			)
@@
 		)
 	)
-	(gr_text "G"
-		(at 121.158 61.722 0)
+	(gr_text "GND"
+		(at 121.158 61.468 0)
 		(layer "F.SilkS")
 		(effects
 			(font
-				(size 1 1)
+				(size 0.6 0.6)
 				(thickness 0.1)
 			)
@@
 		(effects
 			(font
-				(size 1 1)
+				(size 0.6 0.6)
 				(thickness 0.1)
 			)
@@
 	)
 	(gr_text "F power"
-		(at 140.97 76.2 90)
+		(at 139.7 78.994 90)
 		(layer "F.SilkS")
 		(effects
@@
 				(thickness 0.1)
 			)
-			(justify top)
+			(justify right)
 		)
 	)
@@
 		(effects
 			(font
-				(size 1 1)
+				(size 0.6 0.6)
 				(thickness 0.1)
 			)
@@
 	)
 	(gr_text "D power"
-		(at 113.03 76.2 -90)
+		(at 114.3 73.406 270)
 		(layer "F.SilkS")
 		(effects
@@
 				(thickness 0.1)
 			)
-			(justify top)
+			(justify right)
 		)
 	)
@@
 		)
 	)
-	(gr_text "I2C"
-		(at 128.778 65.024 0)
+	(gr_text "i2c"
+		(at 128.778 65.786 0)
 		(layer "F.SilkS")
 		(effects
 			(font
-				(size 1 1)
+				(size 0.6 0.6)
 				(thickness 0.1)
 			)
-			(justify top)
 		)
 	)
@@
 	)
 	(segment
-		(start 117.308 63.46)
-		(end 117.308 62.314168)
+		(start 117.455 61.869)
+		(end 116.586 62.738)
 		(width 0.254)
 		(layer "F.Cu")
@@
 	)
 	(segment
-		(start 117.753168 61.869)
-		(end 127.142 61.869)
+		(start 124.998 76.804192)
+		(end 127 74.802192)
 		(width 0.254)
 		(layer "F.Cu")
@@
 	(segment
 		(start 127.142 61.869)
-		(end 128.773 63.5)
-		(width 0.254)
-		(layer "F.Cu")
-		(net 41)
-	)
-	(segment
-		(start 116.586 62.738)
-		(end 117.308 63.46)
-		(width 0.254)
-		(layer "F.Cu")
-		(net 41)
-	)
-	(segment
-		(start 124.998 76.804192)
-		(end 127 74.802192)
+		(end 117.455 61.869)
 		(width 0.254)
 		(layer "F.Cu")
@@
 	)
 	(segment
-		(start 117.308 62.314168)
-		(end 117.753168 61.869)
+		(start 128.773 63.5)
+		(end 127.142 61.869)
 		(width 0.254)
 		(layer "F.Cu")
@@
 		(polygon
 			(pts
-				(xy 76.2 50.8) (xy 177.8 50.8) (xy 177.8 127) (xy 76.2 127)
+				(xy 88.9 58.42) (xy 165.1 58.42) (xy 165.1 109.22) (xy 88.9 109.22)
 			)
 		)
